File: photovision-boards.kicad_sch (KiCad schematic)
At the start: 0 parts

Commit message: Placed the proccessor
Parts:
- added U1: W65C816SxPL, Package_LCC:PLCC-44, symbol PCM_65xx-library:W65C816SxPL
Connections:
- new net: U1.1 (VSS), U1.23 (VSS), U1.24 (VSS)
- new net: U1.37 (VDD), U1.9 (VDD)
Changed lines of the file:
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@@
 	(generator_version "9.0")
 	(paper "A4")
+	(symbol
+		(lib_id "PCM_65xx-library:W65C816SxPL")
+		(at 43.18 54.61 0)
+		(unit 1)
+		(exclude_from_sim no)
+		(in_bom yes)
+		(on_board yes)
+		(dnp no)
+		(fields_autoplaced yes)
+		(property "Reference" "U1"
+			(at 45.3233 13.97 0)
+			(effects
+				(font
+					(size 1.27 1.27)
+				)
+				(justify left)
+			)
+		)
+		(property "Value" "W65C816SxPL"
+			(at 45.3233 16.51 0)
+			(effects
+				(font
+					(size 1.27 1.27)
+				)
+				(justify left)
+			)
+		)
+		(property "Footprint" "Package_LCC:PLCC-44"
+			(at 43.18 3.81 0)
+			(effects
+				(font
+					(size 1.27 1.27)
+				)
+				(hide yes)
+			)
+		)
+		(property "Datasheet" "http://www.westerndesigncenter.com/wdc/documentation/w65c816s.pdf"
+			(at 43.18 6.35 0)
+			(effects
+				(font
+					(size 1.27 1.27)
+				)
+				(hide yes)
+			)
+		)
+		(property "Description" "8/16-bit CMOS General Purpose Microprocessor, PLCC-44"
+			(at 43.18 54.61 0)
+			(effects
+				(font
+					(size 1.27 1.27)
+				)
+				(hide yes)
+			)
+		)
+		(pin "29"
+		)
+		(pin "16"
+		)
+		(pin "22"
+		)
+		(pin "18"
+		)
+		(pin "19"
+		)
+		(pin "17"
+		)
+		(pin "4"
+		)
+		(pin "15"
+		)
+		(pin "30"
+		)
+		(pin "35"
+		)
+		(pin "7"
+		)
+		(pin "5"
+		)
+		(pin "3"
+		)
+		(pin "38"
+		)
+		(pin "2"
+		)
+		(pin "36"
+		)
+		(pin "25"
+		)
+		(pin "27"
+		)
+		(pin "33"
+		)
+		(pin "44"
+		)
+		(pin "21"
+		)
+		(pin "32"
+		)
+		(pin "34"
+		)
+		(pin "28"
+		)
+		(pin "26"
+		)
+		(pin "31"
+		)
+		(pin "20"
+		)
+		(pin "40"
+		)
+		(pin "12"
+		)
+		(pin "9"
+		)
+		(pin "6"
+		)
+		(pin "37"
+		)
+		(pin "11"
+		)
+		(pin "10"
+		)
+		(pin "8"
+		)
+		(pin "14"
+		)
+		(pin "39"
+		)
+		(pin "24"
+		)
+		(pin "13"
+		)
+		(pin "43"
+		)
+		(pin "42"
+		)
+		(pin "23"
+		)
+		(pin "1"
+		)
+		(pin "41"
+		)
+		(instances
+			(project ""
+				(path "/dca9d465-b063-455c-8145-6543fdb9063c"
+					(reference "U1")
+					(unit 1)
+				)
+			)
+		)
+	)
 	(sheet_instances
 		(path "/"
